File: RX-2040.kicad_sch (KiCad schematic)
At the start: 2 parts, among them P1 USB_C_Plug_USB2.0, U1 RP2350B

Commit message: Cap and Res
Parts:
- removed P1: USB_C_Plug_USB2.0, symbol Connector:USB_C_Plug_USB2.0
- added C1, C10, C11, C13, C14, C15, C20, C21, C27, C4, C5, C6, C7, C8: 100nf, symbol Device:C_Small
- added C12, C19, C2, C26, C3, C9: 2.2uf, symbol Device:C_Small
- added C16, C17, C18, C22: 10uf, symbol Device:C_Small
- added C23, C25, C28, C29, C30, C31, C32, C33, C34, C36: C_Small, symbol Device:C_Small
- added C24, C35: 10pf, symbol Device:C_Small
- added L1: L_Small, symbol Device:L_Small
- added R1, R2, R8: 27r4, symbol Device:R_Small
- added R10: 470r, symbol Device:R_Small
- added R11: 10k, symbol Device:R_Small
- added R12, R24, R25: 100k, symbol Device:R_Small
- added R13, R4, R6: 1k, symbol Device:R_Small
- added R14, R15, R7, R9: 5k1, symbol Device:R_Small
- added R16, R17, R21: R_Small, symbol Device:R_Small
- added R18, R23: 4k7, symbol Device:R_Small
- added R19: 1m5, symbol Device:R_Small
- added R20: 750k, symbol Device:R_Small
- added R22: 100r, symbol Device:R_Small
- added R3: 220r, symbol Device:R_Small
- added R5: 8m06, symbol Device:R_Small
Connections:
- net at U1.10 (DVDD), U1.32 (DVDD), U1.51 (DVDD): now also U1.65 (VREG_FB), C1.2, C18.2, C4.2, C5.2, L1.2
- net at U1.15 (IOVDD), U1.24 (IOVDD), U1.29 (IOVDD)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: now also U1.64 (VREG_VIN), U1.68 (USB_OTP_VDD), U1.69 (QSPI_IOVDD)
- net at U1.63 (VREG_LX): now also L1.1
- new net GND: C1.1, C18.1, C4.1, C5.1
Other:
- moved on the sheet: U1
